Commit message: Update AUBO polish control system

File: src/aubo_robot/aubo_description/urdf/aubo_e5.xacro (robot description, xacro)
@@ -482,4 +482,9 @@
       </geometry>
     </visual>
+    <collision>
+      <geometry>
+        <mesh filename="package://aubo_description/meshes/aubo_e5/collision/pedestal.STL" />
+      </geometry>
+    </collision>
   </link>
   <joint name="pedestal_joint" type="fixed">

File: src/aubo_robot/aubo_gazebo/urdf/aubo_e5.xacro (robot description, xacro)
@@ -308,4 +308,9 @@
       </geometry>
     </visual>
+    <collision>
+      <geometry>
+        <mesh filename="package://aubo_description/meshes/aubo_e5/collision/pedestal.STL" />
+      </geometry>
+    </collision>
   </link>
   <joint name="pedestal_joint" type="fixed">
